File: ESP32_D1_Mini_Breakout/ESP32_D1_Mini_Breakout.brd (EAGLE design)
At the start: 86 x 58 mm, 44 parts, among them U1 ESP32_D1_MINI, X1 5V, X2 3.3V, X3 GND, X4 RESET, X6 ESP32-JTAGTH

Commit message: Done routing Add Gerber files
Parts:
- removed U$2: (no value), M2M-Connectors:1X10-2.54
- added X7: (no value), M2M-Connectors:1X10-2.54
- D1: value (none) -> RED
- D10: value RED -> (none)
- D11: value GREEN -> (none)
- D2: value (none) -> GREEN
- X1: value 5V -> RESET; device M2M-Connectors:1X05-2.54 -> M2M-Switches:TACT-SWITCH-EVQ
- X2: value 3.3V -> (none); device M2M-Connectors:1X05-2.54 -> M2M-Connectors:2X05-1.27-SWD
- X3: value GND -> 5V
- X4: value RESET -> 3.3V; device M2M-Switches:TACT-SWITCH-EVQ -> M2M-Connectors:1X05-2.54
- X5: value (none) -> GND; device M2M-Connectors:1X10-2.54 -> M2M-Connectors:1X05-2.54
- X6: value ESP32-JTAGTH -> (none); device M2M-Connectors:2X05-1.27-SWD -> M2M-Connectors:1X10-2.54
- moved X2 73.1 mm to (79.1, 27.0), turned to 180 degrees
- moved X5 66.0 mm to (6.35, 26.7), turned to 0 degrees
- moved D2 45.5 mm to (20.3, 34.3), turned to 0 degrees
- moved D1 43.8 mm to (20.3, 41.9), turned to 0 degrees
- moved D10 42.2 mm to (62.2, 36.8), turned to 180 degrees
- moved D11 41.9 mm to (62.2, 34.3), turned to 180 degrees
- moved U$4 32.0 mm to (50.8, 8.79)
- moved U$3 31.5 mm to (12.5, 1.54)
- moved X6 28.4 mm to (72.4, 54.6), turned to 270 degrees
- moved X1 25.5 mm to (8.89, 16.5)
- moved X4 18.0 mm to (6.35, 34.3)
- moved D22 15.2 mm to (62.2, 3.81)
- moved X3 15.2 mm to (6.35, 41.9)
- moved D6 5.08 mm to (62.2, 47.0)
- moved D7 5.08 mm to (62.2, 44.5)
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Connections:
- net 3.3V: now also D2.A, X4.1, X4.2, X4.3, X4.4, X4.5; no longer D11.A, X2.2, X2.3, X2.4, X2.5, X6.1
- net 5V: now also D1.A, X3.1, X3.2, X3.3, X3.4, X3.5; no longer D10.A, X1.1, X1.2, X1.3, X1.4, X1.5
- net GND: now also X1.A, X1.A', X2.3, X2.5, X2.9, X5.1, X5.2, X5.3, X5.4, X5.5; no longer X3.1, X3.2, X3.3, X3.4, X3.5, X4.A, X4.A', X6.3, X6.5, X6.9
- net IO0: now also D3.A, X6.1; no longer D1.A, U$2.1
- net IO16: now also D7.A, X6.5; no longer D5.A, U$2.5
- net IO17: now also D8.A, X6.6; no longer D6.A, U$2.6
- net IO18: now also D9.A, X6.7; no longer D7.A, U$2.7
- net IO19: now also D10.A, X6.8; no longer D8.A, U$2.8
- net IO2: now also D4.A, X6.2; no longer D2.A, U$2.2
- net IO21: now also D11.A, X6.9; no longer D9.A, U$2.9
- net IO22: now also X6.10; no longer U$2.10
- net IO23: now also X7.1; no longer X5.1
- net IO25: now also X7.2; no longer X5.2
- net IO26: now also X7.3; no longer X5.3
- net IO27: now also D16.A, X7.4; no longer D22.A, X5.4
- net IO32: now also D17.A, X7.5; no longer D16.A, X5.5
- net IO33: now also D18.A, X7.6; no longer D17.A, X5.6
- net IO34: now also D19.A, X7.7; no longer D18.A, X5.7
- net IO35: now also D20.A, X7.8; no longer D19.A, X5.8
- net IO4: now also D5.A, X6.3; no longer D3.A, U$2.3
- net IO5: now also D6.A, X6.4; no longer D4.A, U$2.4
- net N$1: now also D2.C; no longer D11.C
- net N$10: now also D10.C; no longer D8.C
- net N$11: now also D11.C; no longer D9.C
- net N$16: now also D16.C; no longer D22.C
- net N$19: now also D18.C; no longer D17.C
- net N$2: now also D1.C; no longer D10.C
- net N$20: now also D17.C; no longer D16.C
- net N$21: now also D19.C; no longer D18.C
- net N$22: now also D20.C; no longer D19.C
- net N$23: now also D21.C; no longer D20.C
- net N$24: now also D22.C; no longer D21.C
- net N$3: now also D6.C; no longer D4.C
- net N$4: now also D5.C; no longer D3.C
- net N$5: now also D4.C; no longer D2.C
- net N$6: now also D3.C; no longer D1.C
- net N$7: now also D7.C; no longer D5.C
- net N$8: now also D8.C; no longer D6.C
- net N$9: now also D9.C; no longer D7.C
- net RST: now also X1.B, X1.B', X2.10; no longer X4.B, X4.B', X6.10
- net RX: now also D22.A, X7.10; no longer D21.A, X5.10
- net TCK: now also X2.4; no longer X6.4
- net TDI: now also X2.8; no longer X6.8
- net TDO: now also X2.6; no longer X6.6
- net TMS: now also X2.2; no longer X6.2
- net TX: now also D21.A, X7.9; no longer D20.A, X5.9
Routing:
- net TMS: track 0.00 -> 89.2 mm, vias 0 -> 3
- net TCK: track 0.00 -> 83.4 mm, vias 0 -> 3
- net RX: track 9.41 -> 92.5 mm, vias 0 -> 1
- net TX: track 9.41 -> 88.3 mm, vias 0 -> 1
- net TDI: track 0.00 -> 76.9 mm, vias 0 -> 3
- net RST: track 61.8 -> 136.9 mm, vias 0 -> 1
- net IO35: track 9.41 -> 81.8 mm, vias 0 -> 3
- net IO33: track 9.41 -> 77.5 mm, vias 0 -> 3
- net IO34: track 9.41 -> 74.7 mm, vias 0 -> 3
- net TDO: track 0.00 -> 61.6 mm, vias 0 -> 3
- net IO26: track 9.41 -> 69.2 mm, vias 0 -> 3
- net IO5: track 9.41 -> 67.3 mm, vias 0 -> 1
- net 3.3V: track 26.6 -> 83.9 mm
- net IO23: track 9.41 -> 61.0 mm, vias 0 -> 3
- net IO19: track 9.41 -> 52.5 mm, vias 0 -> 2
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Other:
- board text added: "2022-08-02"
- board text removed: "2022-07-26"
