File: ESP8266_D1_Mini_Breakout/ESP8266_D1_Mini_Breakout.brd (EAGLE design)
At the start: 76.2 x 58.4 mm, 39 parts, among them X1 5V, X2 3.3V, X3 GND, X4 RESET

Commit message: Done routing Add Gerber files
Parts:
- moved U$3 33.0 mm to (14.0, 2.04)
- moved U$4 26.0 mm to (46.8, 9.29)
Changed lines of the file:
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@@
 </element>
 <element name="X1" library="M2M-Connectors" package="1X05-2.54" value="5V" x="6.35" y="41.91" smashed="yes">
-<attribute name="NAME" x="9.525" y="41.275" size="1.016" layer="51"/>
 <attribute name="NAME" x="5.08" y="43.561" size="1.016" layer="25"/>
 <attribute name="NAME" x="11.43" y="41.91" size="1.27" layer="48" align="center"/>
+<attribute name="NAME" x="9.525" y="41.275" size="1.016" layer="51"/>
 <attribute name="VALUE" x="5.08" y="39.37" size="1.016" layer="27"/>
 </element>
 <element name="X2" library="M2M-Connectors" package="1X05-2.54" value="3.3V" x="6.35" y="34.29" smashed="yes">
-<attribute name="NAME" x="9.525" y="33.655" size="1.016" layer="51"/>
 <attribute name="NAME" x="5.08" y="35.941" size="1.016" layer="25"/>
 <attribute name="NAME" x="11.43" y="34.29" size="1.27" layer="48" align="center"/>
+<attribute name="NAME" x="9.525" y="33.655" size="1.016" layer="51"/>
 <attribute name="VALUE" x="5.08" y="31.75" size="1.016" layer="27"/>
 </element>
 <element name="X3" library="M2M-Connectors" package="1X05-2.54" value="GND" x="6.35" y="26.67" smashed="yes">
-<attribute name="NAME" x="9.525" y="26.035" size="1.016" layer="51"/>
 <attribute name="NAME" x="5.08" y="28.321" size="1.016" layer="25"/>
 <attribute name="NAME" x="11.43" y="26.67" size="1.27" layer="48" align="center"/>
+<attribute name="NAME" x="9.525" y="26.035" size="1.016" layer="51"/>
 <attribute name="VALUE" x="5.08" y="24.13" size="1.016" layer="27"/>
 </element>
@@
 </element>
 <element name="U$2" library="M2M-Connectors" package="1X12-2.54" value="HEADER-1X12-2.54" x="68.58" y="43.18" smashed="yes" rot="R270">
-<attribute name="NAME" x="68.58" y="31.75" size="1.27" layer="48" rot="R270" align="center"/>
 <attribute name="NAME" x="67.945" y="33.655" size="1.016" layer="51" rot="R270"/>
 <attribute name="NAME" x="70.1675" y="44.45" size="1.016" layer="25" rot="R270"/>
+<attribute name="NAME" x="68.58" y="31.75" size="1.27" layer="48" rot="R270" align="center"/>
 <attribute name="VALUE" x="66.04" y="44.45" size="1.016" layer="27" rot="R270"/>
 </element>
@@
 <attribute name="VALUE" x="20.32" y="28.575" size="1.016" layer="27" align="bottom-center"/>
 </element>
-<element name="U$3" library="M2M-Frames" package="BERGDAHL-20MM-TPLACE" value="" x="46.99" y="2.54" smashed="yes"/>
-<element name="U$4" library="M2M-Frames" package="OSHW-8MM-TPLACE" value="" x="20.828" y="10.287" smashed="yes"/>
+<element name="U$3" library="M2M-Frames" package="BERGDAHL-20MM-TPLACE" value="" x="13.99" y="2.04" smashed="yes"/>
+<element name="U$4" library="M2M-Frames" package="OSHW-8MM-TPLACE" value="" x="46.828" y="9.287" smashed="yes"/>
 <element name="D12" library="M2M-LED" package="LED0603" value="" x="59.69" y="17.78" smashed="yes" rot="R180">
 <attribute name="NAME" x="59.69" y="17.78" size="0.4064" layer="51" rot="R180" align="center"/>
